File: kicad/OrganUniversalMCUboard/BoardToBoardComms.kicad_sch (KiCad schematic)
At the start: 10 parts, among them J5 UART, J6 CAN, U5 SN65HVD230

Commit message: Finishing MCU board and lots of chimes updates
Parts:
- removed J6: CAN, symbol Connector_Generic:Conn_01x04
- added CD_U5: 100n, Capacitor_SMD:C_0603_1608Metric, symbol Device:C
- added J6: CAN, Connector_JST:JST_PH_B3B-PH-K_1x03_P2.00mm_Vertical, symbol Connector_Generic:Conn_01x03
- J5: footprint (none) -> Connector_JST:JST_PH_B4B-PH-K_1x04_P2.00mm_Vertical
- JP1: footprint (none) -> Connector_PinHeader_2.54mm:PinHeader_1x02_P2.54mm_Vertical
- RS1: footprint (none) -> Resistor_SMD:R_0603_1608Metric
- RS_UART_RX1: renamed from RS_UART_RX; footprint (none) -> Resistor_SMD:R_0603_1608Metric
- RS_UART_TX1: renamed from RS_UART_TX; footprint (none) -> Resistor_SMD:R_0603_1608Metric
- R_TERM1: renamed from R_TERM; footprint (none) -> Resistor_SMD:R_0603_1608Metric
- SJ_COMM_RX1: renamed from SJ_COMM_RX; footprint (none) -> Jumper:SolderJumper-3_P1.3mm_Open_RoundedPad1.0x1.5mm
- SJ_COMM_TX1: renamed from SJ_COMM_TX; footprint (none) -> Jumper:SolderJumper-3_P1.3mm_Open_RoundedPad1.0x1.5mm
Connections:
- net +3.3V: now also CD_U5.1
- net CANH: now also J6.1 (Pin_1)
- net CANL: now also J6.2 (Pin_2)
- net GND: now also CD_U5.2, J6.3 (Pin_3)
