File: kicad/OrganUniversalMCUboard/OrganUniversalMCUboard.kicad_pcb (KiCad board)
At the start: 2 copper layers, 74.1 x 79.8 mm, 64 parts, among them J1 12-15V IN, J10 5V out, J11 GPIO, J2 EXT 5V In/out, J3 MIDI IN MIDI IN, J5 UART, J6 CAN CAN, J7 I2S I2S, J8 SPI, J9 I2C I2C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

Commit message: Finalized v001 of MCU board for production
Parts:
- removed 5VOutEnable: SolderJumper_2_Open, Jumper:SolderJumper-2_P1.3mm_Open_RoundedPad1.0x1.5mm
- removed CAN Term: CAN Terminator, Connector_PinHeader_2.54mm:PinHeader_1x02_P2.54mm_Vertical
- removed FUSE: MF-MSMF050, Fuse:Fuse_1812_4532Metric
- removed J3 MIDI IN: MIDI IN, Connector_JST:JST_PH_B3B-PH-K_1x03_P2.00mm_Vertical
- removed J6 CAN: CAN, Connector_JST:JST_PH_B3B-PH-K_1x03_P2.00mm_Vertical
- removed J7 I2S: I2S, Connector_IDC:IDC-Header_2x05_P2.54mm_Vertical
- removed J9 I2C: I2C, Connector_JST:JST_PH_B4B-PH-K_1x04_P2.00mm_Vertical
- removed JP3: SJ_THRU_SRC, Jumper:SolderJumper-3_P1.3mm_Open_RoundedPad1.0x1.5mm
- removed MIDI OUT/THRU: MIDI OUTTHRU, Connector_JST:JST_PH_B3B-PH-K_1x03_P2.00mm_Vertical
- removed R10: 100k, Resistor_SMD:R_0603_1608Metric
- removed RS_*: 33R, Resistor_SMD:R_0603_1608Metric
- added F1: MF-MSMF050, Fuse:Fuse_1812_4532Metric, F.Cu at (133.6, 119.6)
- added J3: MIDI IN, Connector_JST:JST_PH_B2B-PH-K_1x02_P2.00mm_Vertical, F.Cu at (135.9, 71.0)
- added J4: MIDI_THRU, Connector_JST:JST_PH_B3B-PH-K_1x03_P2.00mm_Vertical, F.Cu at (136.0, 82.7)
- added J6: CAN, Connector_JST:JST_PH_B3B-PH-K_1x03_P2.00mm_Vertical, F.Cu at (69.9, 89.9)
- added J7: I2S, Connector_IDC:IDC-Header_2x05_P2.54mm_Vertical, F.Cu at (71.0, 60.3)
- added J9: I2C, Connector_JST:JST_PH_B4B-PH-K_1x04_P2.00mm_Vertical, F.Cu at (118.9, 61.0)
- added JP1: CAN Terminator, Connector_PinHeader_2.54mm:PinHeader_1x02_P2.54mm_Vertical, F.Cu at (69.7, 81.5)
- added JP2: SolderJumper_2_Open, Jumper:SolderJumper-2_P1.3mm_Open_RoundedPad1.0x1.5mm, F.Cu at (71.9, 94.2)
- added RS_LATCH1: 33R, Resistor_SMD:R_0603_1608Metric, F.Cu at (79.0, 107.3)
- J1: value 12-15V IN -> VIN (12-15V)
Connections:
- Q1 pad 3: /MIDI/MIDI_OUTTHRU_SINK -> /MIDI/MIDI_THRU_SINK
- R2 pad 1: /MIDI/MIDI_OUTTHRU_P5 -> /MIDI/MIDI_THRU_SINK
- R2 pad 2: /MIDI/MIDI_OUTTHRU_SINK -> /MIDI/MIDI_THRU_P5
- R3 pad 1: /MIDI/DRV_IN -> /MIDI/MIDI_THRU_DRV
- R7 pad 2: /MIDI/MIDI_OUTTHRU_P4 -> /MIDI/MIDI_THRU_P4
Routing:
- net /MIDI/MIDI_THRU_P4: track 0.00 -> 8.55 mm
- net /MIDI/MIDI_OUTTHRU_P4: track 8.55 -> 0.00 mm
- net GND: track 323.1 -> 315.8 mm, vias 113 -> 112
- net /MIDI/MIDI_THRU_P5: track 0.00 -> 7.37 mm
- net /MIDI/MIDI_OUTTHRU_P5: track 6.89 -> 0.00 mm
- net /MIDI/DRV_IN: track 4.40 -> 0.00 mm
- net /MIDI/MIDI_THRU_DRV: track 8.98 -> 12.8 mm
- net /MIDI/MIDI_THRU_SINK: track 0.00 -> 2.83 mm
- net /MIDI_GPIO: track 52.5 -> 50.4 mm
- net /MIDI/MIDI_OUTTHRU_SINK: track 1.54 -> 0.00 mm
