File: kicad/OrganUniversalMCUboard/OrganUniversalMCUboard.kicad_sch (KiCad schematic)
At the start: 25 parts, among them J7 Conn_01x06, J8 SPI, J9 I2C, SW1 SW_DIP_x04, U1 ESP32-S3-DevKitC

Commit message: Finishing MCU board and lots of chimes updates
Parts:
- removed D5: Protection Diode, symbol Device:D
- removed J7: Conn_01x06, symbol Connector_Generic:Conn_01x06
- added J11: GPIO, Connector_PinHeader_2.54mm:PinHeader_2x03_P2.54mm_Vertical, symbol Connector_Generic:Conn_01x06
- added J7: I2S, Connector_IDC:IDC-Header_2x05_P2.54mm_Vertical, symbol Connector_Generic:Conn_01x10
- D2, D3: footprint (none) -> LED_SMD:LED_0603_1608Metric
- J8: footprint (none) -> Connector_IDC:IDC-Header_2x05_P2.54mm_Vertical
- J9: footprint (none) -> Connector_JST:JST_PH_B4B-PH-K_1x04_P2.00mm_Vertical
- JP2: footprint (none) -> Jumper:SolderJumper-2_P1.3mm_Open_RoundedPad1.0x1.5mm
- RLED1, RLED2: footprint (none) -> Resistor_SMD:R_0805_2012Metric
- RP_DIP1, RP_DIP2, RP_DIP3, RP_DIP4: footprint (none) -> Resistor_SMD:R_0603_1608Metric
- RP_SCL1: renamed from RP_SCL; footprint (none) -> Resistor_SMD:R_0603_1608Metric
- RP_SDA1: renamed from RP_SDA; footprint (none) -> Resistor_SMD:R_0603_1608Metric
- RS_BCLK1: renamed from RS_BCLK; footprint (none) -> Resistor_SMD:R_0603_1608Metric
- RS_CLR1: renamed from RS_CLR; footprint (none) -> Resistor_SMD:R_0603_1608Metric
- RS_DIN1: renamed from RS_DIN; footprint (none) -> Resistor_SMD:R_0603_1608Metric
- RS_LATCH1: renamed from RS_LATCH; footprint (none) -> Resistor_SMD:R_0603_1608Metric
- RS_LRCLK1: renamed from RS_LRCLK; footprint (none) -> Resistor_SMD:R_0603_1608Metric
- RS_MOSI1: renamed from RS_MOSI; footprint (none) -> Resistor_SMD:R_0603_1608Metric
- RS_OE_N1: renamed from RS_OE_N; footprint (none) -> Resistor_SMD:R_0603_1608Metric
- RS_SCK1: renamed from RS_SCK; footprint (none) -> Resistor_SMD:R_0603_1608Metric
- SW1: value SW_DIP_x04 -> MODES; footprint (none) -> Button_Switch_THT:SW_DIP_SPSTx04_Slide_6.7x11.72mm_W7.62mm_P2.54mm_LowProfile
Connections:
- net +3.3V: now also J11.1 (Pin_1), J7.1 (Pin_1)
- net COMM_RX: now also U1.9 (GPIO16/ADC2_CH5/32K_N); no longer U1.11 (GPIO18/ADC2_CH7)
- net COMM_TX: now also U1.11 (GPIO18/ADC2_CH7); no longer U1.9 (GPIO16/ADC2_CH5/32K_N)
- net GND: now also J11.2 (Pin_2), J7.2 (Pin_2), J7.3 (Pin_3), J7.8 (Pin_8), J7.9 (Pin_9)
- net I2S_MCLK: now also J7.7 (Pin_7)
- net SYS_5V: now also U1.21 (5V), J7.10 (Pin_10)
- net GPIO8: now reaches U1.12 (GPIO8/ADC1_CH7)
- net GPIO8: now also J11.3 (Pin_3)
- net GPIO9: now reaches U1.15 (GPIO9/ADC1_CH8)
- net GPIO9: now also J11.4 (Pin_4)
- net GPIO37: now reaches U1.34 (GPIO37)
- net GPIO37: now also J11.5 (Pin_5)
- net GPIO38: now reaches U1.35 (GPIO38)
- net GPIO38: now also J11.6 (Pin_6)
- net at RS_BCLK1.1: now also J7.4 (Pin_4)
- net at RS_LRCLK1.1: now also J7.5 (Pin_5)
- net at RS_DIN1.1: now also J7.6 (Pin_6)
- no-connect marks 1 -> 14
Other:
- moved on the sheet: SW1

Commit message: Something...
Parts:
- added J12, J13, J14, J15, J16, J17, J18, J19, J20, J21, J22, J23: Conn_01x01, Connector_PinHeader_2.54mm:PinHeader_1x01_P2.54mm_Vertical, symbol Connector_Generic:Conn_01x01
Connections:
- net at U1.13 (GPIO3/ADC1_CH2): now also J17.1 (Pin_1)
- net at U1.14 (GPIO46): now also J19.1 (Pin_1)
- net at U1.25 (GPIO19/USB_D-): now also J15.1 (Pin_1)
- net at U1.26 (GPIO20/USB_D+): now also J14.1 (Pin_1)
- net at U1.30 (GPIO45): now also J18.1 (Pin_1)
- net at U1.31 (GPIO0): now also J16.1 (Pin_1)
- net at U1.36 (GPIO39/MTCK): now also J20.1 (Pin_1)
- net at U1.37 (GPIO40/MTDO): now also J21.1 (Pin_1)
- net at U1.38 (GPIO41/MTDI): now also J22.1 (Pin_1)
- net at U1.39 (GPIO42/MTMS): now also J23.1 (Pin_1)
- net at U1.42 (GPIO44/U0RXD): now also J13.1 (Pin_1)
- net at U1.43 (GPIO43/U0TXD): now also J12.1 (Pin_1)
- no-connect marks 14 -> 2
