File: kicad/OrganKeyswitchBreakout/breakout_chip.kicad_sch (KiCad schematic)
At the start: 10 parts, among them J1 Conn_01x16, U1 MCP23017_SS

Commit message: Finishing keyswitch breakout board
Parts:
- CD_U1: footprint (none) -> Capacitor_SMD:C_0805_2012Metric
- J1: footprint (none) -> Connector_IDC:IDC-Header_2x08_P2.54mm_Vertical
- JP1, JP2, JP3: footprint (none) -> Jumper:SolderJumper-2_P1.3mm_Bridged_RoundedPad1.0x1.5mm
- R1, R2, R3, R4: footprint (none) -> Resistor_SMD:R_0805_2012Metric
