File: kicad/OrganUnifiedSoundboard/16_channel_mosfet_output.kicad_sch (KiCad schematic)
At the start: 0 parts

Commit message: Finalized unified soundboard driver for production, adding some models
Other:
- sheet mosfet_channel1 ports: added none; removed 12VFlyback
- sheet mosfet_channel10 ports: added none; removed 12VFlyback
- sheet mosfet_channel11 ports: added none; removed 12VFlyback
- sheet mosfet_channel12 ports: added none; removed 12VFlyback
- sheet mosfet_channel13 ports: added none; removed 12VFlyback
- sheet mosfet_channel14 ports: added none; removed 12VFlyback
- sheet mosfet_channel15 ports: added none; removed 12VFlyback
- sheet mosfet_channel16 ports: added none; removed 12VFlyback
- sheet mosfet_channel2 ports: added none; removed 12VFlyback
- sheet mosfet_channel3 ports: added none; removed 12VFlyback
- sheet mosfet_channel4 ports: added none; removed 12VFlyback
- sheet mosfet_channel5 ports: added none; removed 12VFlyback
- sheet mosfet_channel6 ports: added none; removed 12VFlyback
- sheet mosfet_channel7 ports: added none; removed 12VFlyback
- sheet mosfet_channel8 ports: added none; removed 12VFlyback
- sheet mosfet_channel9 ports: added none; removed 12VFlyback
