File: kicad/OrganUnifiedSoundboard/BoardToBoardComms.kicad_sch (KiCad schematic)
At the start: 8 parts, among them J6 CAN, U5 SN65HVD230

Commit message: Adding some custom components that some of the kicad things depend on
Parts:
- added J4: CAN_THRU, Connector_JST:JST_PH_B3B-PH-K_1x03_P2.00mm_Vertical, symbol Connector_Generic:Conn_01x03
Connections:
- net CANH: now also J4.1 (Pin_1)
- net CANL: now also J4.2 (Pin_2)
- net GND: now also J4.3 (Pin_3)
Changed lines of the file:
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@@
 	(paper "A4")
+	(junction
+		(at 161.29 69.85)
+		(diameter 0)
+		(color 0 0 0 0)
+	)
 	(junction
 		(at 129.54 95.25)
@@
 	)
 	(junction
+		(at 162.56 72.39)
+		(diameter 0)
+		(color 0 0 0 0)
+	)
+	(junction
 		(at 146.05 69.85)
 		(diameter 0)
@@
 	(wire
 		(pts
+			(xy 181.61 69.85) (xy 181.61 66.04)
+		)
+		(stroke
+			(width 0)
+			(type default)
+		)
+	)
+	(wire
+		(pts
 			(xy 113.03 95.25) (xy 129.54 95.25)
 		)
@@
 	(wire
 		(pts
-			(xy 146.05 69.85) (xy 167.64 69.85)
-		)
-		(stroke
-			(width 0)
-			(type default)
-		)
-	)
-	(wire
-		(pts
-			(xy 158.75 72.39) (xy 167.64 72.39)
+			(xy 146.05 69.85) (xy 161.29 69.85)
+		)
+		(stroke
+			(width 0)
+			(type default)
+		)
+	)
+	(wire
+		(pts
+			(xy 158.75 72.39) (xy 162.56 72.39)
 		)
 		(stroke
@@
 	(wire
 		(pts
+			(xy 181.61 72.39) (xy 179.07 72.39)
+		)
+		(stroke
+			(width 0)
+			(type default)
+		)
+	)
+	(wire
+		(pts
 			(xy 113.03 80.01) (xy 113.03 83.82)
 		)
@@
 	(wire
 		(pts
-			(xy 162.56 74.93) (xy 167.64 74.93)
+			(xy 162.56 82.55) (xy 162.56 72.39)
+		)
+		(stroke
+			(width 0)
+			(type default)
+		)
+	)
+	(wire
+		(pts
+			(xy 161.29 69.85) (xy 167.64 69.85)
+		)
+		(stroke
+			(width 0)
+			(type default)
+		)
+	)
+	(wire
+		(pts
+			(xy 161.29 66.04) (xy 161.29 69.85)
 		)
 		(stroke
@@
 	(wire
 		(pts
+			(xy 179.07 82.55) (xy 162.56 82.55)
+		)
+		(stroke
+			(width 0)
+			(type default)
+		)
+	)
+	(wire
+		(pts
 			(xy 158.75 72.39) (xy 158.75 87.63)
 		)
@@
 	(wire
 		(pts
+			(xy 181.61 66.04) (xy 161.29 66.04)
+		)
+		(stroke
+			(width 0)
+			(type default)
+		)
+	)
+	(wire
+		(pts
 			(xy 68.58 69.85) (xy 80.01 69.85)
 		)
@@
 	(wire
 		(pts
+			(xy 179.07 72.39) (xy 179.07 82.55)
+		)
+		(stroke
+			(width 0)
+			(type default)
+		)
+	)
+	(wire
+		(pts
 			(xy 139.7 87.63) (xy 139.7 77.47)
 		)
@@
 		(pts
 			(xy 146.05 80.01) (xy 146.05 87.63)
+		)
+		(stroke
+			(width 0)
+			(type default)
+		)
+	)
+	(wire
+		(pts
+			(xy 162.56 72.39) (xy 167.64 72.39)
 		)
 		(stroke
@@
 	)
 	(symbol
+		(lib_id "power:GND")
+		(at 181.61 74.93 0)
+		(unit 1)
+		(exclude_from_sim no)
+		(in_bom yes)
+		(on_board yes)
+		(dnp no)
+		(fields_autoplaced yes)
+		(property "Reference" "#PWR015"
+			(at 181.61 81.28 0)
+			(effects
+				(font
+					(size 1.27 1.27)
+				)
+				(hide yes)
+			)
+		)
+		(property "Value" "GND"
+			(at 181.61 80.01 0)
+			(effects
+				(font
+					(size 1.27 1.27)
+				)
+			)
+		)
+		(property "Footprint" ""
+			(at 181.61 74.93 0)
+			(effects
+				(font
+					(size 1.27 1.27)
+				)
+				(hide yes)
+			)
+		)
+		(property "Datasheet" ""
+			(at 181.61 74.93 0)
+			(effects
+				(font
+					(size 1.27 1.27)
+				)
+				(hide yes)
+			)
+		)
+		(property "Description" "Power symbol creates a global label with name \"GND\" , ground"
+			(at 181.61 74.93 0)
+			(effects
+				(font
+					(size 1.27 1.27)
+				)
+				(hide yes)
+			)
+		)
+		(pin "1"
+		)
+		(instances
+			(project "OrganUnifiedSoundboard"
+				(path "/4a899aa1-9bb8-4bd0-98b8-a923f79fe9df/cfa6cbaf-d0e0-41c4-8de8-02a89a1099b2/82107bef-a801-4c3d-ac88-a6fb788da9b1"
+					(reference "#PWR015")
+					(unit 1)
+				)
+			)
+		)
+	)
+	(symbol
+		(lib_id "Connector_Generic:Conn_01x03")
+		(at 186.69 72.39 0)
+		(unit 1)
+		(exclude_from_sim no)
+		(in_bom yes)
+		(on_board yes)
+		(dnp no)
+		(fields_autoplaced yes)
+		(property "Reference" "J4"
+			(at 189.23 71.1199 0)
+			(effects
+				(font
+					(size 1.27 1.27)
+				)
+				(justify left)
+			)
+		)
+		(property "Value" "CAN_THRU"
+			(at 189.23 73.6599 0)
+			(effects
+				(font
+					(size 1.27 1.27)
+				)
+				(justify left)
+			)
+		)
+		(property "Footprint" "Connector_JST:JST_PH_B3B-PH-K_1x03_P2.00mm_Vertical"
+			(at 186.69 72.39 0)
+			(effects
+				(font
+					(size 1.27 1.27)
+				)
+				(hide yes)
+			)
+		)
+		(property "Datasheet" "~"
+			(at 186.69 72.39 0)
+			(effects
+				(font
+					(size 1.27 1.27)
+				)
+				(hide yes)
+			)
+		)
+		(property "Description" "Generic connector, single row, 01x03, script generated (kicad-library-utils/schlib/autogen/connector/)"
+			(at 186.69 72.39 0)
+			(effects
+				(font
+					(size 1.27 1.27)
+				)
+				(hide yes)
+			)
+		)
+		(pin "1"
+		)
+		(pin "3"
+		)
+		(pin "2"
+		)
+		(instances
+			(project "OrganUnifiedSoundboard"
+				(path "/4a899aa1-9bb8-4bd0-98b8-a923f79fe9df/cfa6cbaf-d0e0-41c4-8de8-02a89a1099b2/82107bef-a801-4c3d-ac88-a6fb788da9b1"
+					(reference "J4")
+					(unit 1)
+				)
+			)
+		)
+	)
+	(symbol
 		(lib_id "Device:R_Small_US")
 		(at 113.03 86.36 0)
@@
 	(symbol
 		(lib_id "power:GND")
-		(at 162.56 74.93 0)
+		(at 167.64 74.93 0)
 		(unit 1)
 		(exclude_from_sim no)
@@
 		(fields_autoplaced yes)
 		(property "Reference" "#PWR018"
-			(at 162.56 81.28 0)
+			(at 167.64 81.28 0)
 			(effects
 				(font
@@
 		)
 		(property "Value" "GND"
-			(at 162.56 80.01 0)
+			(at 167.64 80.01 0)
 			(effects
 				(font
@@
 		)
 		(property "Footprint" ""
-			(at 162.56 74.93 0)
+			(at 167.64 74.93 0)
 			(effects
 				(font
@@
 		)
 		(property "Datasheet" ""
-			(at 162.56 74.93 0)
+			(at 167.64 74.93 0)
 			(effects
 				(font
@@
 		)
 		(property "Description" "Power symbol creates a global label with name \"GND\" , ground"
-			(at 162.56 74.93 0)
-			(effects
-				(font
+			(at 167.64 74.93 0)
+			(effects
+				(font

Commit message: Finalized unified soundboard driver for production, adding some models
Parts:
- JP1: value CAN Terminator -> CAN Term?
Changed lines of the file:
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@@
 			)
 		)
-		(property "Value" "CAN Terminator"
+		(property "Value" "CAN Term?"
 			(at 147.32 73.6599 90)
 			(effects
