File: kicad/OrganUnifiedSoundboard/MIDI.kicad_sch (KiCad schematic)
At the start: 15 parts, among them J1 SDS-50J, J3 SDS-50J, Q1 MMBT3904, Q2 MMBT3904, U2 6N137

Commit message: Adding some custom components that some of the kicad things depend on
Parts:
- J1, J3: footprint CONN5_SDS-50J_CUD -> CustomLibrary:Custom_CONN5_SDS-50J_CUD
Changed lines of the file:
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@@
 			)
 		)
-		(property "Footprint" "CONN5_SDS-50J_CUD"
+		(property "Footprint" "CustomLibrary:Custom_CONN5_SDS-50J_CUD"
 			(at 219.71 99.06 0)
 			(effects
@@
 			)
 		)
-		(property "Footprint" "CONN5_SDS-50J_CUD"
+		(property "Footprint" "CustomLibrary:Custom_CONN5_SDS-50J_CUD"
 			(at 104.14 33.02 0)
 			(effects
